File: alf_board_v8.brd (EAGLE design)
At the start: 230 x 140.6 mm, 194 parts, among them CN1 СНП15-48, IC12 YM2149F / AY-3-8910, IC13 ALS138/1533ID7, IC14 ALS00/1533LA3, IC16 ALS93/1533IE5, IC17 74HC595, IC18 74HC595, IC19 7493 / 155IE5, IC2 ALS240 / 1533AP3, IC20 ALS04/1533LN1, IC21 ALS251/1533KP15, IC22 CXA1645, IC23 74HCT04, IC5 ALS09/1533LI2, IC6 LS245 / 555AP6, J1 2.1MMJACKTHM, Q1 8Mhz, Q2 14Mhz, Q3 4,433619Mhz, X1 RCA_L, X2 RCA_R, X3 RGB-OUT, X4 JOY-1, X5 JOY-2, X6 Video, X7 s-video, X8 SCART-F

Commit message: vil0
Parts:
- removed C10, C11, C12, C13, C14, C15, C16, C17, C18, C19, C20, C21, C3, C44, C45, C46, C9: (no value), rcl:C0805
- removed H2, H3, H4: MOUNT-PAD-ROUND3.3, holes:3,3-PAD
- removed H5, H6: MOUNT-PAD-ROUND3.2, holes:3,2-PAD
- removed JP1: (no value), pinhead:1X03
- removed KD6: (no value), pinhead:1X01
- removed SJ1: (no value), jumper:SJ_2
- added /RES, A0, A1, A10, A11, A12, A13, A14, A15, A2, A3, A4, A5, A6, A7, A8, A9, AR0, AR1, AR2, AR3, AR4, AR5, AR6, AR7, BUSAK, BUSRQ, CE, DB0, DB1, DB2, DB3, DB4, DB5, DB6, DB7, DR0, DR1, DR2, DR3, DR4, DR5, DR6, DR7, INT, IORQ, KA10, KA11, KA12, KA13, KA14, KA15, KA8, KA9, M1, MREQ, NMI, RD, RES, RFSH, ROM, SSWR, WAIT, WR: (no value), pinhead:1X01
- added D10, D11, D4, D5, D6, D7, D8, D9: LL4148, diode:SOD80C
- added IC1: 74HC00N, 74xx-eu:DIL14
- added JP1A, JP1A1: (no value), pinhead:1X03
- added JP1B, JPORT: (no value), jumper:SJ_2
- added ROMCE: (no value), jumper:SJ
- added TI, TO: (no value), pinhead:1X02
- C4: device rcl:C0805 -> rcl:C102-043X133
- DD2: value Z80A -> Z80
- DD4: value T34VG1 -> Т34ВГ1
- IC6: device 74xx-eu:DIL20 -> 74xx-eu:SO20W
- R23: device rcl:R0805 -> rcl:0207/12
- R24: device rcl:R0805 -> rcl:0207/10
- moved IC13 545.7 mm to (-92.9, -228.7)
- moved IC14 530.2 mm to (-76.0, -234.1), turned to 270 degrees
- moved IC16 482.4 mm to (-73.2, -209.3), turned to 90 degrees
- moved IC12 472.2 mm to (-55.4, -219.5), turned to 270 degrees
- moved C5 467.9 mm to (-70.2, -184.9)
- moved C7 467.9 mm to (-45.7, -161.3)
- moved C8 467.9 mm to (-63.4, -161.4)
- moved R28 467.9 mm to (-51.5, -156.8)
- moved R29 467.9 mm to (-46.2, -168.1)
- moved R35 467.9 mm to (-68.4, -168.1)
- moved R37 467.9 mm to (-62.9, -168.1)
- moved R30 467.9 mm to (-40.8, -168.1)
- moved R31 467.9 mm to (-51.5, -162.2)
- moved R32 467.9 mm to (-51.5, -168.1)
- moved R33 467.9 mm to (-57.5, -162.2)
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Connections:
- net /CAS renamed !CAS
- net /RAS renamed !RAS
- net /WE renamed !WE
- net BR renamed Y
- net N$12 renamed R_INT
- net N$76 renamed CAS_RAM
- net N$77 renamed RAS_RAM
- removed net /BUSAK: CN1.11
- removed net /BUSRQ: CN1.9, DD2.25, R14.2
- removed net /CE: DD4.36, DD8.2, DD8.4, IC5.1
- removed net /INT: CN1.19, DD2.16, R25.2
- removed net /IORQ: CN1.7, DD2.20, DD4.23, IC13.4
- removed net /M1: CN1.40, DD2.27, DD4.22, IC13.6
- removed net /MREQ: CN1.5, DD2.19, DD4.28
- removed net /NMI: CN1.23, DD2.17, R13.2
- removed net /RD: CN1.42, DD2.21, DD4.29
- removed net /RFSH: CN1.46, DD2.28, DD4.24
- removed net /SSRD: CN1.17, DD4.27, DD8.13, IC5.2
- removed net /SSWR: CN1.43, DD4.26, DD8.9
- removed net /WAIT: CN1.21, DD2.24, DD4.34
- removed net /WR: CN1.44, DD2.22, DD4.25, IC13.1
- new net !BUSAK: BUSAK.1, DD2.23
- new net !BUSRQ: BUSRQ.1, DD2.25, R14.2
- new net !CE: CE.1, DD4.36, ROMCE.2
- new net !INT: DD2.16, INT.1, R25.2
- new net !IORQ: DD2.20, DD4.23, IORQ.1
- new net !M1: DD2.27, DD4.22, M1.1
- new net !MREQ: DD2.19, DD4.28, MREQ.1
- new net !NMI: DD2.17, NMI.1, R13.2
- new net !RD: DD2.21, DD4.29, RD.1
- new net !RFSH: DD2.28, DD4.24, RFSH.1
- new net !SSRD: DD4.27, JP1A1.3, JPORT.1
- new net !SSWR: DD4.26, SSWR.1
- new net !WAIT: DD2.24, DD4.34, WAIT.1
- new net !WR: DD2.22, DD4.25, WR.1
- new net DD7Q2: DD7.7, JP1A.1, JP1B.3
- new net N$100: IC6.1, JP1A1.2, JPORT.2
- new net N$93: D5.A, KA9.1
- new net N$94: D6.A, KA10.1
- new net N$95: D7.A, KA11.1
- new net N$96: D8.A, KA12.1
- new net N$97: D9.A, KA13.1
- new net N$98: D10.A, KA14.1
- new net N$99: D11.A, KA15.1
- new net TAPE_IN: DD4.19, TI.2
- new net TAPE_OUT: DD4.13, TO.2
- new net VCC: DD7.16, DD8.14, IC1.14, IC13.16, IC14.14, IC17.16, IC18.16, IC19.5, IC2.20, IC20.14, IC21.16, IC23.14, IC5.14, IC6.20
- new net _!CE: DD8.2, DD8.4, IC5.1
- new net _!IORQ: IC13.4
- new net _!M1: IC13.6
- new net _!RES: IC12.23
- new net _!ROM: DD8.3
- new net _!SSRD: DD8.13, IC5.2
- new net _!SSWR: DD8.9
- new net _!WR: IC13.1
- new net _1IC8: IC5.3, IC5.6, R4.2
- new net _A1: DD1.11, IC13.5
- new net _A14: IC13.2
- new net _A15: IC13.3
- new net _DB0: IC12.37
- new net _DB1: IC12.36
- new net _DB2: IC12.35
- new net _DB3: IC12.34
- new net _DB4: IC12.33
- new net _DB5: IC12.32
- new net _DB6: IC12.31
- new net _DB7: IC12.30
- new net _TO: IC12.21
- net !RES: now also /RES.1, IC1.6; no longer CN1.38, DD1.8, IC12.23
- net !ROM: now also ROM.1, ROMCE.1; no longer CN1.3, DD8.3
- net !ROMC: no longer CN1.15
- net +5V: now also JP1A.3, JP1B.1; no longer C10.2, C11.2, C12.2, C13.2, C14.2, C15.2, C16.2, C17.2, C18.2, C19.2, C20.2, C21.2, C44.2, C45.2, C46.2, C9.2, DD7.16, DD8.14, IC13.16, IC14.14, IC17.16, IC18.16, IC19.5, IC2.20, IC20.14, IC21.16, IC23.14, IC5.14, IC6.20, JP1.3
- net 1IC8: now also JP1A1.1, JPORT.3; no longer CN1.31, IC5.3, IC5.6, IC6.1, R4.2
- net 8M: now also IC1.11; no longer DD1.4
- net A0: now also A0.1; no longer CN1.4
- net A1: now also A1.1; no longer CN1.6, DD1.11, IC13.5
- net A10: now also A10.1, D6.C; no longer CN1.24
- net A11: now also A11.1, D7.C; no longer CN1.26
- net A12: now also A12.1, D8.C; no longer CN1.28
- net A13: now also A13.1, D9.C; no longer CN1.30
- net A14: now also A14.1, D10.C; no longer CN1.32, IC13.2
- net A15: now also A15.1, D11.C; no longer CN1.34, IC13.3
- net A2: now also A2.1; no longer CN1.8
- net A3: now also A3.1; no longer CN1.10
- net A4: now also A4.1; no longer CN1.12
- net A5: now also A5.1; no longer CN1.14
- net A6: now also A6.1; no longer CN1.16
- net A7: now also A7.1; no longer CN1.18
- net A8: now also A8.1, D4.C; no longer CN1.20
- net A9: now also A9.1, D5.C; no longer CN1.22
- net AR0: now also AR0.1
- net AR1: now also AR1.1
- net AR2: now also AR2.1
- net AR3: now also AR3.1
- net AR4: now also AR4.1
- net AR5: now also AR5.1
- net AR6: now also AR6.1
- net AR7: now also AR7.1
- net B1: now also JP1A.2, JP1B.2; no longer JP1.2
- net DB0: now also DB0.1; no longer CN1.27, IC12.37
- net DB1: now also DB1.1; no longer CN1.29, IC12.36
- net DB2: now also DB2.1; no longer CN1.25, IC12.35
- net DB3: now also DB3.1; no longer CN1.36, IC12.34
- net DB4: now also DB4.1; no longer CN1.35, IC12.33
- net DB5: now also DB5.1; no longer CN1.37, IC12.32
- net DB6: now also DB6.1; no longer CN1.39, IC12.31
- net DB7: now also DB7.1; no longer CN1.41, IC12.30
- net DR0: now also DR0.1
- net DR1: now also DR1.1
- net DR2: now also DR2.1
- net DR3: now also DR3.1
- net DR4: now also DR4.1
- net DR5: now also DR5.1
- net DR6: now also DR6.1
- net DR7: now also DR7.1
- net GND: now also IC1.7; no longer C10.1, C11.1, C12.1, C13.1, C14.1, C15.1, C16.1, C17.1, C18.1, C19.1, C20.1, C21.1, C44.1, C45.1, C46.1, C9.1, H1.B3,3, H2.B3,3, H3.B3,3, H4.B3,3, H5.B3,2, H6.B3,2
- net KD6: now also TI.1; no longer DD4.19, KD6.1
- net N$2: now also IC1.8; no longer DD1.2
- net N$3: now also IC1.12, IC1.13; no longer DD1.3
- net N$37: now also IC14.6
- net N$38: now also IC14.1, IC14.2
- net N$39: now also IC14.3
- net N$4: now also IC1.10, IC1.9; no longer DD1.1
- net N$40: now also IC14.4, IC14.5
- net N$8: now also IC1.1, IC1.2; no longer DD1.5
- net N$9: now also D4.A, KA8.1; no longer DD7.7, JP1.1
- net PBANK: no longer CN1.13
- net RES: now also IC1.3, IC1.4, IC1.5, RES.1; no longer CN1.45, DD1.6, DD1.9
- net SOUND-IN: no longer CN1.33
- net TO: now also TO.1; no longer DD4.13, IC12.21
Routing:
- net /MREQ: track 176.2 -> 0.00 mm, vias 4 -> 0
- net DB7: track 199.9 -> 36.4 mm, vias 6 -> 0
- net DR4: track 32.4 -> 193.6 mm
- net DB6: track 193.5 -> 35.6 mm, vias 5 -> 0
- net DR6: track 0.00 -> 153.0 mm, vias 0 -> 3
- net /IORQ: track 140.0 -> 0.00 mm, vias 3 -> 0
- net !RES: track 135.5 -> 0.00 mm, vias 4 -> 0
- net DR2: track 0.00 -> 132.9 mm, vias 0 -> 4
- net +5V: track 352.0 -> 219.5 mm, vias 8 -> 4
- net DR5: track 66.8 -> 196.4 mm, vias 2 -> 4
- net A14: track 130.5 -> 2.22 mm, vias 7 -> 0
- net DR0: track 0.00 -> 120.0 mm, vias 0 -> 4
- net /NMI: track 109.1 -> 0.00 mm, vias 4 -> 0
- net DB2: track 109.4 -> 7.62 mm, vias 5 -> 0
- net A9: track 146.3 -> 45.3 mm, vias 5 -> 0
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Other:
- board size 230 x 140.6 mm -> 214.1 x 128.6 mm

Commit message: ..
Parts:
- added D12: LL4148, diode:SOD80C
Connections:
- net +5V: now also D12.C
- net N$8: now also D12.A
