File: alf_board_v8.sch (EAGLE design)
At the start: 192 parts, among them CN1 СНП15-48, IC12 YM2149F / AY-3-8910, IC13 ALS138/1533ID7, IC14 ALS00/1533LA3, IC16 ALS93/1533IE5, IC17 74HC595, IC18 74HC595, IC19 7493 / 155IE5, IC2 ALS240 / 1533AP3, IC20 ALS04/1533LN1, IC21 ALS251/1533KP15, IC22 CXA1645, IC23 74HCT04, IC5 ALS09/1533LI2, IC6 LS245 / 555AP6, J1 2.1MMJACKTHM, Q1 8Mhz, Q2 14Mhz, Q3 4,433619Mhz, X1 RCA_L, X2 RCA_R, X3 RGB-OUT, X4 JOY-1, X5 JOY-2, X6 Video, X7 s-video, X8 SCART-F

Commit message: vil0
Parts:
- removed C10, C11, C12, C13, C14, C15, C16, C17, C18, C19, C20, C21, C3, C44, C45, C46, C9: (no value), rcl:C-EUC0805
- removed H2, H3, H4: MOUNT-PAD-ROUND3.3, holes:MOUNT-PAD-ROUND3.3
- removed H5, H6: MOUNT-PAD-ROUND3.2, holes:MOUNT-PAD-ROUND3.2
- removed JP1: (no value), pinhead:PINHD-1X3
- removed KD6: (no value), pinhead:PINHD-1X1
- removed SJ1: (no value), jumper:SJ2W
- added /RES, A0, A1, A10, A11, A12, A13, A14, A15, A2, A3, A4, A5, A6, A7, A8, A9, AR0, AR1, AR2, AR3, AR4, AR5, AR6, AR7, BUSAK, BUSRQ, CE, DB0, DB1, DB2, DB3, DB4, DB5, DB6, DB7, DR0, DR1, DR2, DR3, DR4, DR5, DR6, DR7, INT, IORQ, KA10, KA11, KA12, KA13, KA14, KA15, KA8, KA9, M1, MREQ, NMI, RD, RES, RFSH, ROM, SSWR, WAIT, WR: (no value), pinhead:PINHD-1X1
- added D10, D11, D4, D5, D6, D7, D8, D9: LL4148, diode:DIODE-SOD80C
- added IC1: 74HC00N, 74xx-eu:74HC00N
- added JP1A, JP1A1: (no value), pinhead:PINHD-1X3
- added JP1B, JPORT: (no value), jumper:SJ2W
- added ROMCE: (no value), jumper:SJ
- added TI, TO: (no value), pinhead:PINHD-1X2
- C4: device rcl:C-EUC0805 -> rcl:C-EU102-043X133
- DD2: value Z80A -> Z80; OC_FARNELL unknown -> (none)
- DD3: MPN (none) -> AT27C020-90PU; OC_NEWARK (none) -> 68T4266; PACKAGE (none) -> PDIP-32; SUPPLIER (none) -> ATMEL
- DD4: value T34VG1 -> Т34ВГ1; OC_FARNELL unknown -> (none)
- DD5, DD6: OC_FARNELL unknown -> (none)
- IC6: device 74xx-eu:74LS245N -> 74xx-eu:74LS245DW
- R23: device rcl:R-EU_R0805 -> rcl:R-EU_0207/12
- R24: device rcl:R-EU_R0805 -> rcl:R-EU_0207/10
Connections:
- net /CAS renamed !CAS
- net /RAS renamed !RAS
- net /WE renamed !WE
- net BR renamed Y
- net N$12 renamed R_INT
- net N$76 renamed CAS_RAM
- net N$77 renamed RAS_RAM
- removed net /BUSAK: CN1.11
- removed net /BUSRQ: CN1.9, DD2.BUSRQ, R14.2
- removed net /CE: DD4.36, DD8A.I1, DD8B.I0, IC5A.I0
- removed net /INT: CN1.19, DD2.INT, R25.2
- removed net /IORQ: CN1.7, DD2.IORQ, DD4.23, IC13A.G2A
- removed net /M1: CN1.40, DD2.M1, DD4.22, IC13A.G1
- removed net /MREQ: CN1.5, DD2.MREQ, DD4.28
- removed net /NMI: CN1.23, DD2.NMI, R13.2
- removed net /RD: CN1.42, DD2.RD, DD4.29
- removed net /RFSH: CN1.46, DD2.RFSH, DD4.24
- removed net /SSRD: CN1.17, DD4.27, DD8D.I1, IC5A.I1
- removed net /SSWR: CN1.43, DD4.26, DD8C.I0
- removed net /WAIT: CN1.21, DD2.WAIT, DD4.34
- removed net /WR: CN1.44, DD2.WR, DD4.25, IC13A.A
- new net !BUSAK: BUSAK.1, DD2.BUSAK
- new net !BUSRQ: BUSRQ.1, DD2.BUSRQ, R14.2
- new net !CE: CE.1, DD4.36, ROMCE.2
- new net !INT: DD2.INT, INT.1, R25.2
- new net !IORQ: DD2.IORQ, DD4.23, IORQ.1
- new net !M1: DD2.M1, DD4.22, M1.1
- new net !MREQ: DD2.MREQ, DD4.28, MREQ.1
- new net !NMI: DD2.NMI, NMI.1, R13.2
- new net !RD: DD2.RD, DD4.29, RD.1
- new net !RFSH: DD2.RFSH, DD4.24, RFSH.1
- new net !SSRD: DD4.27, JP1A1.3, JPORT.1
- new net !SSWR: DD4.26, SSWR.1
- new net !WAIT: DD2.WAIT, DD4.34, WAIT.1
- new net !WR: DD2.WR, DD4.25, WR.1
- new net DD7Q2: DD7A.Q2, JP1A.1, JP1B.3
- new net N$100: IC6A.DIR, JP1A1.2, JPORT.2
- new net N$93: D5.A, KA9.1
- new net N$94: D6.A, KA10.1
- new net N$95: D7.A, KA11.1
- new net N$96: D8.A, KA12.1
- new net N$97: D9.A, KA13.1
- new net N$98: D10.A, KA14.1
- new net N$99: D11.A, KA15.1
- new net TAPE_IN: DD4.19, TI.2
- new net TAPE_OUT: DD4.13, TO.2
- new net _!CE: DD8A.I1, DD8B.I0, IC5A.I0
- new net _!IORQ: IC13A.G2A
- new net _!M1: IC13A.G1
- new net _!RES: IC12.!RESET
- new net _!ROM: DD8A.O
- new net _!SSRD: DD8D.I1, IC5A.I1
- new net _!SSWR: DD8C.I0
- new net _!WR: IC13A.A
- new net _1IC8: IC5A.O, IC5B.O, R4.2
- new net _A1: DD1E.I, IC13A.G2B
- new net _A14: IC13A.B
- new net _A15: IC13A.C
- new net _DB0: IC12.DA0
- new net _DB1: IC12.DA1
- new net _DB2: IC12.DA2
- new net _DB3: IC12.DA3
- new net _DB4: IC12.DA4
- new net _DB5: IC12.DA5
- new net _DB6: IC12.DA6
- new net _DB7: IC12.DA7
- new net _TO: IC12.IOA0
- net !RES: now also /RES.1, IC1B.O; no longer CN1.38, DD1D.O, IC12.!RESET
- net !ROM: now also ROM.1, ROMCE.1; no longer CN1.3, DD8A.O
- net !ROMC: no longer CN1.15
- net +5V: now also JP1A.3, JP1B.1; no longer C10.2, C11.2, C12.2, C13.2, C14.2, C15.2, C16.2, C17.2, C18.2, C19.2, C20.2, C21.2, C44.2, C45.2, C46.2, C9.2, DD7P.VCC, DD8P.VCC, IC13P.VCC, IC14P.VCC, IC17P.VCC, IC18P.VCC, IC19P.VCC, IC20P.VCC, IC21P.VCC, IC23P.VCC, IC2P.VCC, IC5P.VCC, IC6P.VCC, JP1.3
- net 1IC8: now also JP1A1.1, JPORT.3; no longer CN1.31, IC5A.O, IC5B.O, IC6A.DIR, R4.2
- net 8M: now also IC1D.O; no longer DD1B.O
- net A0: now also A0.1; no longer CN1.4
- net A1: now also A1.1; no longer CN1.6, DD1E.I, IC13A.G2B
- net A10: now also A10.1, D6.C; no longer CN1.24
- net A11: now also A11.1, D7.C; no longer CN1.26
- net A12: now also A12.1, D8.C; no longer CN1.28
- net A13: now also A13.1, D9.C; no longer CN1.30
- net A14: now also A14.1, D10.C; no longer CN1.32, IC13A.B
- net A15: now also A15.1, D11.C; no longer CN1.34, IC13A.C
- net A2: now also A2.1; no longer CN1.8
- net A3: now also A3.1; no longer CN1.10
- net A4: now also A4.1; no longer CN1.12
- net A5: now also A5.1; no longer CN1.14
- net A6: now also A6.1; no longer CN1.16
- net A7: now also A7.1; no longer CN1.18
- net A8: now also A8.1, D4.C; no longer CN1.20
- net A9: now also A9.1, D5.C; no longer CN1.22
- net AR0: now also AR0.1
- net AR1: now also AR1.1
- net AR2: now also AR2.1
- net AR3: now also AR3.1
- net AR4: now also AR4.1
- net AR5: now also AR5.1
- net AR6: now also AR6.1
- net AR7: now also AR7.1
- net B1: now also JP1A.2, JP1B.2; no longer JP1.2
- net DB0: now also DB0.1; no longer CN1.27, IC12.DA0
- net DB1: now also DB1.1; no longer CN1.29, IC12.DA1
- net DB2: now also DB2.1; no longer CN1.25, IC12.DA2
- net DB3: now also DB3.1; no longer CN1.36, IC12.DA3
- net DB4: now also DB4.1; no longer CN1.35, IC12.DA4
- net DB5: now also DB5.1; no longer CN1.37, IC12.DA5
- net DB6: now also DB6.1; no longer CN1.39, IC12.DA6
- net DB7: now also DB7.1; no longer CN1.41, IC12.DA7
- net DR0: now also DR0.1
- net DR1: now also DR1.1
- net DR2: now also DR2.1
- net DR3: now also DR3.1
- net DR4: now also DR4.1
- net DR5: now also DR5.1
- net DR6: now also DR6.1
- net DR7: now also DR7.1
- net GND: no longer C10.1, C11.1, C12.1, C13.1, C14.1, C15.1, C16.1, C17.1, C18.1, C19.1, C20.1, C21.1, C44.1, C45.1, C46.1, C9.1, DD7P.GND, DD8P.GND, H1.MOUNT, H2.MOUNT, H3.MOUNT, H4.MOUNT, H5.MOUNT, H6.MOUNT, IC13P.GND, IC14P.GND, IC17P.GND, IC18P.GND, IC19P.GND, IC20P.GND, IC21P.GND, IC23P.GND, IC2P.GND, IC5P.GND, IC6P.GND
- net KD6: now also TI.1; no longer DD4.19, KD6.1
- net N$2: now also IC1C.O; no longer DD1A.O
- net N$3: now also IC1D.I0, IC1D.I1; no longer DD1B.I
- net N$37: now also IC14B.O
- net N$38: now also IC14A.I0, IC14A.I1
- net N$39: now also IC14A.O
- net N$4: now also IC1C.I0, IC1C.I1; no longer DD1A.I
- net N$40: now also IC14B.I0, IC14B.I1
- net N$8: now also IC1A.I0, IC1A.I1; no longer DD1C.I
- net N$9: now also D4.A, KA8.1; no longer DD7A.Q2, JP1.1
- net PBANK: no longer CN1.13
- net RES: now also IC1A.O, IC1B.I0, IC1B.I1, RES.1; no longer CN1.45, DD1C.O, DD1D.I
- net SOUND-IN: no longer CN1.33
- net TO: now also TO.1; no longer DD4.13, IC12.IOA0
Other:
- note added: "RAM"
- note added: "КА1515ХМ1-216"
- note added: "нет пинов PBANK !ROMC SOUND-IN"
- moved on the sheet: B0, B1, B2, B3, C1, C2, C22, C23, C24, C25, C26, C27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

Commit message: ..
Parts:
- added D12: LL4148, diode:DIODE-SOD80C
Connections:
- net +5V: now also D12.C
- net N$8: now also D12.A
Changed lines of the file:
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@@
 <part name="ROMCE" library="jumper" deviceset="SJ" device=""/>
 <part name="IC1" library="74xx-eu" deviceset="74*00" device="N" technology="HC"/>
+<part name="D12" library="diode" deviceset="DIODE-" device="SOD80C" value="LL4148"/>
 </parts>
 <sheets>
@@
 <attribute name="VALUE" x="264.922" y="82.55" size="1.778" layer="96" rot="R90"/>
 </instance>
-<instance part="P+2" gate="1" x="261.62" y="96.52"/>
+<instance part="P+2" gate="1" x="266.7" y="93.98" smashed="yes" rot="R270">
+<attribute name="VALUE" x="269.24" y="93.98" size="1.778" layer="96"/>
+</instance>
 <instance part="GND2" gate="1" x="261.62" y="63.5"/>
 <instance part="P+3" gate="1" x="566.42" y="530.86" smashed="yes">
@@
 <instance part="GND13" gate="1" x="335.28" y="408.94" rot="R270"/>
 <instance part="S1" gate="1" x="254" y="71.12" smashed="yes">
-<attribute name="NAME" x="248.92" y="90.17" size="1.778" layer="95" rot="R180"/>
-<attribute name="VALUE" x="249.555" y="85.09" size="1.778" layer="96"/>
+<attribute name="NAME" x="251.46" y="67.31" size="1.778" layer="95" rot="R180"/>
+<attribute name="VALUE" x="244.475" y="59.69" size="1.778" layer="96"/>
 </instance>
 <instance part="CN1" gate="G$1" x="665.48" y="584.2">
@@
 <instance part="IC1" gate="C" x="335.28" y="78.74"/>
 <instance part="IC1" gate="D" x="373.38" y="78.74"/>
+<instance part="D12" gate="G$1" x="254" y="86.36" smashed="yes" rot="R90">
+<attribute name="NAME" x="248.92" y="88.4174" size="1.778" layer="95" rot="R180"/>
+<attribute name="VALUE" x="248.92" y="86.1314" size="1.778" layer="96" rot="R180"/>
+</instance>
 </instances>
 <busses>
@@
 <pinref part="R3" gate="G$1" pin="2"/>
 <pinref part="P+2" gate="1" pin="+5V"/>
-<wire x1="261.62" y1="91.44" x2="261.62" y2="93.98" width="0.1524" layer="91"/>
+<wire x1="264.16" y1="93.98" x2="261.62" y2="93.98" width="0.1524" layer="91"/>
+<wire x1="261.62" y1="93.98" x2="261.62" y2="91.44" width="0.1524" layer="91"/>
+<wire x1="261.62" y1="93.98" x2="254" y2="93.98" width="0.1524" layer="91"/>
+<pinref part="D12" gate="G$1" pin="C"/>
+<wire x1="254" y1="93.98" x2="254" y2="88.9" width="0.1524" layer="91"/>
+<junction x="261.62" y="93.98"/>
 </segment>
 <segment>
@@
 <wire x1="266.7" y1="81.28" x2="264.16" y2="81.28" width="0.1524" layer="91"/>
 <junction x="264.16" y="78.74"/>
+<pinref part="D12" gate="G$1" pin="A"/>
+<wire x1="254" y1="83.82" x2="254" y2="78.74" width="0.1524" layer="91"/>
 </segment>
 </net>
